Commit message: first draft of model composition
need validators to generate a valid urdf

File: examples/test_kin_xtext/src-gen/demo.urdf (robot description, URDF)
Before this commit: robot ur5, 2 links, 1 joints
Links:
- removed link base_link
- added link dummy_link
Joints:
- removed joint shoulder_pan_joint
- added joint combination_joint: type None, parent base_link, child shoulder_link
