Commit message: generate cylinder geometry

File: examples/generated/test_macro.xacro (robot description, xacro)
@@ -6,8 +6,10 @@
 			<visual>
 				<geometry>
+					<cylinder length="0.04" radius"0.1"/>
 				</geometry>
 			</visual>
 			<collision>
 				<geometry>
+					<cylinder length="0.04" radius"0.1"/>
 				</geometry>
 			</collision>
