Commit message: add limits to revolute joints

File: examples/generated/PiTasc/kr16_2_macro.xacro (robot description, xacro)
@@ -145,5 +145,6 @@
 			<child link="${prefix}link_1" />
 			<origin xyz="0 0 0.675" rpy="0 0 0" />
-			<axis xyz="0 0 -1">
+			<axis xyz="0 0 -1" />
+			<limit effort="0" lower="${radians(-185)}" upper="${radians(185)}" velocity="${radians(156)}" />
 		</joint>
 		<joint name="${prefix}joint_a2" type="revolute">
@@ -151,5 +152,6 @@
 			<child link="${prefix}link_2" />
 			<origin xyz="0.26 0 0" rpy="0 0 0" />
-			<axis xyz="0 1 0">
+			<axis xyz="0 1 0" />
+			<limit effort="0" lower="${radians(-155)}" upper="${radians(35)}" velocity="${radians(156)}" />
 		</joint>
 		<joint name="${prefix}joint_a3" type="revolute">
@@ -157,5 +159,6 @@
 			<child link="${prefix}link_3" />
 			<origin xyz="0.68 0 0" rpy="0 0 0" />
-			<axis xyz="0 1 0">
+			<axis xyz="0 1 0" />
+			<limit effort="0" lower="${radians(-130)}" upper="${radians(154)}" velocity="${radians(156)}" />
 		</joint>
 		<joint name="${prefix}joint_a4" type="revolute">
@@ -163,5 +166,6 @@
 			<child link="${prefix}link_4" />
 			<origin xyz="0.67 0 -0.035" rpy="0 0 0" />
-			<axis xyz="-1 0 0">
+			<axis xyz="-1 0 0" />
+			<limit effort="0" lower="${radians(-350)}" upper="${radians(350)}" velocity="${radians(330)}" />
 		</joint>
 		<joint name="${prefix}joint_a5" type="revolute">
@@ -169,5 +173,6 @@
 			<child link="${prefix}link_5" />
 			<origin xyz="0 0 0" rpy="0 0 0" />
-			<axis xyz="0 1 0">
+			<axis xyz="0 1 0" />
+			<limit effort="0" lower="${radians(-130)}" upper="${radians(130)}" velocity="${radians(330)}" />
 		</joint>
 		<joint name="${prefix}joint_a6" type="revolute">
@@ -175,4 +180,5 @@
 			<child link="${prefix}link_6" />
 			<origin xyz="0 0 0.675" rpy="0 0 0" />
+			<limit effort="0" lower="${radians(-350)}" upper="${radians(350)}" velocity="${radians(615)}" />
 		</joint>
 		<joint name="${prefix}joint_a6_flange" type="revolute">
