Commit message: fix errors in PiTasc example

File: examples/PiTasc/ati_axia80.xacro (robot description, xacro)
@@ -10,5 +10,5 @@
 					Link { name "prefix"robotside
 						visual Visual {
-							origin Pose { rpy "0 0 0" xyz "0 ${pi} 0" }
+							origin Pose { rpy "0 ${pi} 0" xyz "0 0 0" }
 							geometry Geometry {
 								mesh Mesh {
@@ -26,5 +26,5 @@
 						parent "prefixrobotside"
 						child "prefixtoolside"
-						origin Pose { rpy "0 0 0.0254" xyz "0 0 0" } },
+						origin Pose { rpy "0 0 0" xyz "0 0 0.0254" } },
 					Joint { name "prefix"measurement_joint
 						type fixed

File: examples/PiTasc/axia80_adapter_plates.xacro (robot description, xacro)
@@ -50,5 +50,10 @@
 			body Body {
 				link {
-					Link { name axia80_adapter_toolside_sensor },
+					Link { name axia80_adapter_toolside_sensor
+						visual Visual {
+							origin Pose { rpy "${pi} 0 ${pi}" xyz "0 0 0" }
+							geometry Geometry {
+								mesh Mesh {
+									filename "package://schrauber_description/mesh/Aufnahme_FT_Sensor_Werkzeugseite_origin.STL" } } } },
 					Link { name axia80_adapter_toolside_changer_sensor } }
 				joint {
@@ -56,10 +61,10 @@
 						type fixed
 						parent parent_link
-						child "axia80_adapter_toolside_changer_sensor"
+						child "axia80_adapter_toolside_sensor"
 						origin "origin_joint" },
 					Joint { name axia80_adapter_toolside_sensor_changer_joint
 						type fixed
 						parent "axia80_adapter_toolside_sensor"
-						child "axia80_adapter_robotside_changer_sensor"
+						child "axia80_adapter_toolside_changer_sensor"
 						origin Pose { rpy "0 0 0" xyz "0 0 0.01" } } } } } }
 }

File: examples/PiTasc/kr16_2_macro.xacro (robot description, xacro)
@@ -140,19 +140,19 @@
 						parent "prefixlink_5"
 						child "prefixlink_6"
-						origin Pose { rpy "0 0 0" xyz "0 0 0.675" }
+						origin Pose { rpy "0 0 0" xyz "0 0 0" }
+						axis Vector3 { xyz "-1 0 0" }
 						limit Limit { effort "0" lower "${radians(-350)}" upper "${radians(350)}" velocity "${radians(615)}" } },
 					Joint { name "prefix"joint_a6_flange
-						type revolute
+						type fixed
 						parent "prefixlink_6"
 						child "prefixflange"
-						origin Pose { rpy "0 0 0" xyz "0.158 0 0" }
-						axis Vector3 { xyz "-1 0 0" } },
+						origin Pose { rpy "0 0 0" xyz "0.158 0 0" } },
 					Joint { name "prefix"base_link_base
-						type revolute
+						type fixed
 						parent "prefixbase_link"
 						child "prefixbase"
-						origin Pose { rpy "0 0 0" xyz "0 0 0.675" } },
+						origin Pose { rpy "0 0 0" xyz "0 0 0" } },
 					Joint { name "prefix"flange_tool0
-						type revolute
+						type fixed
 						parent "prefixflange"
 						child "prefixtool0"

File: examples/generated/PiTasc/ati_axia80.xacro (robot description, xacro)
@@ -4,4 +4,5 @@
 		<link name="${prefix}robotside" >
 			<visual>
+				<origin xyz="0 0 0" rpy="0 ${pi} 0" />"
 				<geometry>
 					<mesh filename="package://ati_force_sensor/urdf/mesh/ATI-9105-Axia80-M20.stl" />
@@ -15,15 +16,15 @@
 		<joint name="${prefix}robotside_joint" type="fixed">
 			<parent link="${parent_link}" />
-			<child link="ati_axia80_robotside" />
+			<child link="${prefix}robotside" />
 			<xacro:insert_block name="origin_joint"/>
 		</joint>
 		<joint name="${prefix}toolside_joint" type="fixed">
-			<parent link="ati_axia80_robotside" />
-			<child link="ati_axia80_toolside" />
-			<origin xyz="0 0 0" rpy="0 0 0.0254" />
+			<parent link="${prefix}robotside" />
+			<child link="${prefix}toolside" />
+			<origin xyz="0 0 0.0254" rpy="0 0 0" />
 		</joint>
 		<joint name="${prefix}measurement_joint" type="fixed">
-			<parent link="ati_axia80_toolside" />
-			<child link="ati_axia80_force_sensor_frame" />
+			<parent link="${prefix}toolside" />
+			<child link="${prefix}force_sensor_frame" />
 			<origin xyz="0 0 0" rpy="0 0 0" />
 		</joint>

File: examples/generated/PiTasc/axia80_adapter_plates.xacro (robot description, xacro)
@@ -20,4 +20,5 @@
 		<link name="axia80_adapter_robotside_changer_sensor" >
 			<visual>
+				<origin xyz="0 0 0" rpy="0 0 0" />"
 				<geometry>
 					<mesh filename="package://schrauber_description/mesh/Aufnahme_FT_Sensor_origin.STL" />
@@ -40,4 +41,10 @@
 	<xacro:macro name="axia80_adapter_toolside_sensor" params="parent_link *origin_joint ">
 		<link name="axia80_adapter_toolside_sensor" >
+			<visual>
+				<origin xyz="0 0 0" rpy="${pi} 0 ${pi}" />"
+				<geometry>
+					<mesh filename="package://schrauber_description/mesh/Aufnahme_FT_Sensor_Werkzeugseite_origin.STL" />
+				</geometry>
+			</visual>
 		</link>
 		<link name="axia80_adapter_toolside_changer_sensor" >
@@ -45,10 +52,10 @@
 		<joint name="axia80_adapter_toolside_sensor_joint" type="fixed">
 			<parent link="${parent_link}" />
-			<child link="axia80_adapter_toolside_changer_sensor" />
+			<child link="axia80_adapter_toolside_sensor" />
 			<xacro:insert_block name="origin_joint"/>
 		</joint>
 		<joint name="axia80_adapter_toolside_sensor_changer_joint" type="fixed">
 			<parent link="axia80_adapter_toolside_sensor" />
-			<child link="axia80_adapter_robotside_changer_sensor" />
+			<child link="axia80_adapter_toolside_changer_sensor" />
 			<origin xyz="0 0 0.01" rpy="0 0 0" />
 		</joint>

File: examples/generated/PiTasc/kr16.urdf (robot description, URDF)
Before this commit: robot kr16, 21 links, 20 joints
Links:
- link axia80_adapter_toolside_sensor: geometry visual mesh filename=package://schrauber_description/mesh/Aufnahme_FT_Sensor_Wer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
Joints:
- joint ati_axia80_toolside_joint: origin xyz=0 0 0 rpy=0 0 0.0254 -> xyz=0 0 0.0254 rpy=0 0 0
- joint axia80_adapter_toolside_sensor_changer_joint: child axia80_adapter_robotside_changer_sensor -> axia80_adapter_toolside_changer_sensor
- joint axia80_adapter_toolside_sensor_joint: child axia80_adapter_toolside_changer_sensor -> axia80_adapter_toolside_sensor
- joint kr16_base_link_base: origin xyz=0 0 0.675 rpy=0 0 0 -> xyz=0 0 0 rpy=0 0 0; type revolute -> fixed
- joint kr16_flange_tool0: type revolute -> fixed
- joint kr16_joint_a1: limit (none) -> lower=-3.2288591161895095 upper=3.2288591161895095 effort=0 velocity=2.722713633111154
- joint kr16_joint_a2: limit (none) -> lower=-2.705260340591211 upper=0.6108652381980153 effort=0 velocity=2.722713633111154
- joint kr16_joint_a3: limit (none) -> lower=-2.2689280275926285 upper=2.6878070480712677 effort=0 velocity=2.722713633111154
- joint kr16_joint_a4: limit (none) -> lower=-6.1086523819801535 upper=6.1086523819801535 effort=0 velocity=5.759586531581287
- joint kr16_joint_a5: limit (none) -> lower=-2.2689280275926285 upper=2.2689280275926285 effort=0 velocity=5.759586531581287
- joint kr16_joint_a6: axis (none) -> -1 0 0; limit (none) -> lower=-6.1086523819801535 upper=6.1086523819801535 effort=0 velocity=10.733774899765127; origin xyz=0 0 0.675 rpy=0 0 0 -> xyz=0 0 0 rpy=0 0 0
- joint kr16_joint_a6_flange: axis -1 0 0 -> (none); type revolute -> fixed

File: examples/generated/PiTasc/kr16_2_macro.xacro (robot description, xacro)
@@ -4,4 +4,5 @@
 		<link name="${prefix}base_link" >
 			<visual>
+				<origin xyz="0 0 0" rpy="0 0 0" />"
 				<geometry>
 					<mesh filename="package://kuka_kr16_support/meshes/kr16_2/visual/base_link.dae" />
@@ -9,4 +10,5 @@
 			</visual>
 			<collision>
+				<origin xyz="0 0 0" rpy="0 0 0" />"
 				<geometry>
 					<mesh filename="package://kuka_kr16_support/meshes/kr16_2/collision/base_link.stl" />
@@ -14,5 +16,5 @@
 			</collision>
 			<inertial>
-				<mass value="2.0">
+				<mass value="2.0" />
 				<origin xyz="0 0 0" rpy="0 0 0" />
 				<inertia ixx="0.01" ixy="0.0" ixz="0.0"
@@ -23,4 +25,5 @@
 		<link name="${prefix}link_1" >
 			<visual>
+				<origin xyz="0 0 0" rpy="0 0 0" />"
 				<geometry>
 					<mesh filename="package://kuka_kr16_support/meshes/kr16_2/visual/link_1.dae" />
@@ -28,4 +31,5 @@
 			</visual>
 			<collision>
+				<origin xyz="0 0 0" rpy="0 0 0" />"
 				<geometry>
 					<mesh filename="package://kuka_kr16_support/meshes/kr16_2/collision/link_1.stl" />
@@ -33,5 +37,5 @@
 			</collision>
 			<inertial>
-				<mass value="2.0">
+				<mass value="2.0" />
 				<origin xyz="0 0 0" rpy="0 0 0" />
 				<inertia ixx="0.01" ixy="0.0" ixz="0.0"
@@ -42,4 +46,5 @@
 		<link name="${prefix}link_2" >
 			<visual>
+				<origin xyz="0 0 0" rpy="0 0 0" />"
 				<geometry>
 					<mesh filename="package://kuka_kr16_support/meshes/kr16_2/visual/link_2.dae" />
@@ -47,4 +52,5 @@
 			</visual>
 			<collision>
+				<origin xyz="0 0 0" rpy="0 0 0" />"
 				<geometry>
 					<mesh filename="package://kuka_kr16_support/meshes/kr16_2/collision/link_2.stl" />
@@ -52,5 +58,5 @@
 			</collision>
 			<inertial>
-				<mass value="2.0">
+				<mass value="2.0" />
 				<origin xyz="0 0 0" rpy="0 0 0" />
 				<inertia ixx="0.01" ixy="0.0" ixz="0.0"
@@ -61,4 +67,5 @@
 		<link name="${prefix}link_3" >
 			<visual>
+				<origin xyz="0 0 0" rpy="0 0 0" />"
 				<geometry>
 					<mesh filename="package://kuka_kr16_support/meshes/kr16_2/visual/link_3.dae" />
@@ -66,4 +73,5 @@
 			</visual>
 			<collision>
+				<origin xyz="0 0 0" rpy="0 0 0" />"
 				<geometry>
 					<mesh filename="package://kuka_kr16_support/meshes/kr16_2/collision/link_3.stl" />
@@ -71,5 +79,5 @@
 			</collision>
 			<inertial>
-				<mass value="2.0">
+				<mass value="2.0" />
 				<origin xyz="0 0 0" rpy="0 0 0" />
 				<inertia ixx="0.01" ixy="0.0" ixz="0.0"
@@ -80,4 +88,5 @@
 		<link name="${prefix}link_4" >
 			<visual>
+				<origin xyz="0 0 0" rpy="0 0 0" />"
 				<geometry>
 					<mesh filename="package://kuka_kr16_support/meshes/kr16_2/visual/link_4.dae" />
@@ -85,4 +94,5 @@
 			</visual>
 			<collision>
+				<origin xyz="0 0 0" rpy="0 0 0" />"
 				<geometry>
 					<mesh filename="package://kuka_kr16_support/meshes/kr16_2/collision/link_4.stl" />
@@ -90,5 +100,5 @@
 			</collision>
 			<inertial>
-				<mass value="2.0">
+				<mass value="2.0" />
 				<origin xyz="0 0 0" rpy="0 0 0" />
 				<inertia ixx="0.01" ixy="0.0" ixz="0.0"
@@ -99,4 +109,5 @@
 		<link name="${prefix}link_5" >
 			<visual>
+				<origin xyz="0 0 0" rpy="0 0 0" />"
 				<geometry>
 					<mesh filename="package://kuka_kr16_support/meshes/kr16_2/visual/link_5.dae" />
@@ -104,4 +115,5 @@
 			</visual>
 			<collision>
+				<origin xyz="0 0 0" rpy="0 0 0" />"
 				<geometry>
 					<mesh filename="package://kuka_kr16_support/meshes/kr16_2/collision/link_5.stl" />
@@ -109,5 +121,5 @@
 			</collision>
 			<inertial>
-				<mass value="2.0">
+				<mass value="2.0" />
 				<origin xyz="0 0 0" rpy="0 0 0" />
 				<inertia ixx="0.01" ixy="0.0" ixz="0.0"
@@ -118,4 +130,5 @@
 		<link name="${prefix}link_6" >
 			<visual>
+				<origin xyz="0 0 0" rpy="0 0 0" />"
 				<geometry>
 					<mesh filename="package://kuka_kr16_support/meshes/kr16_2/visual/link_6.dae" />
@@ -123,4 +136,5 @@
 			</visual>
 			<collision>
+				<origin xyz="0 0 0" rpy="0 0 0" />"
 				<geometry>
 					<mesh filename="package://kuka_kr16_support/meshes/kr16_2/collision/link_6.stl" />
@@ -128,5 +142,5 @@
 			</collision>
 			<inertial>
-				<mass value="2.0">
+				<mass value="2.0" />
 				<origin xyz="0 0 0" rpy="0 0 0" />
 				<inertia ixx="0.01" ixy="0.0" ixz="0.0"
@@ -179,19 +193,19 @@
 			<parent link="${prefix}link_5" />
 			<child link="${prefix}link_6" />
-			<origin xyz="0 0 0.675" rpy="0 0 0" />
+			<origin xyz="0 0 0" rpy="0 0 0" />
+			<axis xyz="-1 0 0" />
 			<limit effort="0" lower="${radians(-350)}" upper="${radians(350)}" velocity="${radians(615)}" />
 		</joint>
-		<joint name="${prefix}joint_a6_flange" type="revolute">
+		<joint name="${prefix}joint_a6_flange" type="fixed">
 			<parent link="${prefix}link_6" />
 			<child link="${prefix}flange" />
 			<origin xyz="0.158 0 0" rpy="0 0 0" />
-			<axis xyz="-1 0 0">
-		</joint>
-		<joint name="${prefix}base_link_base" type="revolute">
+		</joint>
+		<joint name="${prefix}base_link_base" type="fixed">
 			<parent link="${prefix}base_link" />
 			<child link="${prefix}base" />
-			<origin xyz="0 0 0.675" rpy="0 0 0" />
-		</joint>
-		<joint name="${prefix}flange_tool0" type="revolute">
+			<origin xyz="0 0 0" rpy="0 0 0" />
+		</joint>
+		<joint name="${prefix}flange_tool0" type="fixed">
 			<parent link="${prefix}flange" />
 			<child link="${prefix}tool0" />
